File: picostation_pcb.kicad_pcb (KiCad board)
At the start: 2 copper layers, 54.5 x 83.1 mm, 67 parts, among them J1 USB_C_Receptacle_USB2.0, J2 +, J3 D, J4 C, J5 G, J6 Conn_01x20, SW1 BOOT, U1 LM78M05_TO252, U3 RP2040, U4 W25Q16JVSSIQ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

Commit message: Updated Board
 * removed SD-Cart Clock PullUp
 * added Active-LED (untested)
 * added Run PullUp
Parts:
- added D1: LED, LED_SMD:LED_0805_2012Metric_Pad1.15x1.40mm_HandSolder, F.Cu at (186.5, 48.5)
- added R29: 2.2k, Resistor_SMD:R_0603_1608Metric_Pad0.98x0.95mm_HandSolder, F.Cu at (190.6, 48.5)
- added R30: 10k, Resistor_SMD:R_0603_1608Metric_Pad0.98x0.95mm_HandSolder, F.Cu at (216.8, 92.8)
- R16: value 100R -> 47R
- moved D2 1.58 mm to (186.5, 46.4)
- moved R2 1.58 mm to (190.6, 46.4)
Connections:
- U3 pad 26: +3V3 -> Net-(U3-RUN)
Routing:
- net SD_MISO: track 24.6 -> 68.7 mm
- net Net-(U3-RUN): track 0.00 -> 8.57 mm
- net +3V3: track 27.1 -> 23.7 mm
- net Net-(D1-A): track 0.00 -> 2.13 mm
- net +5V: track 51.3 -> 53.3 mm
- net GP18: track 32.9 -> 33.0 mm, vias 0 -> 2
Other:
- board text added: "ACTIVE"
- board text added: "v20230513"
- board text removed: "v20230502"
